File: adventure-board.kicad_sch (KiCad schematic)
At the start: 361 parts, among them J1 BreadboardHdr_2x10, J2 Conn_01x05, J4 HY2.0-4P-WT, J5 HY2.0-4P-WT, SW1 SW_MEC_5G, SW2 SW_MEC_5G, SW3 SW_MEC_5G, SW4 SW_MEC_5G, SW5 SW_MEC_5G, SW6 SW_MEC_5G, SW7 BOOTSEL, SW8 RESET, U1 RP2350A, U10 IS31FL3729, U11 IS31FL3729, U2 H5VHD3BC, U3 GT-USB-7010ASV, U4 W25Q64JVSSIQ, U6 PESD5V0U2BT, U7 TPS2065CDBV, U8 PAM8302AASCR, U9 AMS1117-3.3, Y1 12MHz

Commit message: Fix 'Staus' typo in schematic, drop reorder steps from README
Regenerate the schematic PDFs with kicad-cli 9.0.

Co-Authored-By: Claude Opus 5.5 <noreply@anthropic.com>
Other:
- note added: "Status LED"
- note removed: "Staus LED"
Changed lines of the file:
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@@
 		)
 	)
-	(text "Staus LED\n"
+	(text "Status LED\n"
 		(exclude_from_sim no)
 		(at 147.066 190.246 0)
